File: laboratorio_1/Cad/laboratorio1.kicad_pcb (KiCad board)
At the start: 2 copper layers, 31 parts, among them J5 Output, U1 TL084, U2 TL084, j1 Vdd, j2 Vss, j3 GND, j4 Input

Commit message: ahora si actualizo con windows el kicad
Parts:
- R11, R12: value R -> 1k
- moved R1 86.5 mm to (115.7, 125.1)
- moved R2 86.3 mm to (115.5, 110.0)
- moved U1 81.5 mm to (135.3, 110.0)
- moved U2 79.6 mm to (154.9, 110.0)
- moved R12 78.7 mm to (178.0, 137.4), turned to 180 degrees
- moved C1 78.5 mm to (130.2, 120.5), turned to -90 degrees
- moved R11 75.2 mm to (179.9, 122.1), turned to -90 degrees
- moved C2 70.3 mm to (130.2, 115.0), turned to 90 degrees
- moved R9 70.0 mm to (162.2, 131.9)
- moved R15 65.8 mm to (174.4, 125.3), turned to 90 degrees
- moved R5 63.8 mm to (115.5, 132.0)
- moved R6 62.3 mm to (129.2, 132.0)
- moved R10 58.7 mm to (139.2, 140.0)
- moved R14 55.9 mm to (154.1, 140.0)
- moved C3 54.8 mm to (168.2, 115.1), turned to -90 degrees
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Routing:
- net Net-(U1E-V+): track 0.00 -> 261.0 mm
- net Net-(U1E-V-): track 0.00 -> 109.4 mm
- net Net-(J5-In): track 0.00 -> 98.1 mm
- net Net-(U1C-+): track 0.00 -> 69.8 mm
- net Net-(U2A--): track 0.00 -> 62.4 mm
- net Net-(R3-Pad2): track 0.00 -> 50.6 mm
- net Net-(j4-In): track 0.00 -> 34.8 mm
- net Net-(U1A--): track 0.00 -> 33.8 mm
- net Net-(C4-Pad2): track 0.00 -> 33.2 mm
- net Net-(U2C--): track 0.00 -> 32.7 mm
- net Net-(C3-Pad2): track 0.00 -> 22.9 mm
- net Net-(C1-Pad2): track 0.00 -> 22.6 mm
- net Net-(U1B--): track 0.00 -> 18.4 mm
- net Net-(C2-Pad2): track 0.00 -> 16.6 mm
- net Net-(U2D-+): track 0.00 -> 11.9 mm
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- added copper zone on B.Cu, net GND
Other:
- board outline added: 93.5 x 96 mm
- board text added: "R5"

Commit message: ggregue Jumper al Cad
Parts:
- added J6: VA1, Connector_PinHeader_1.00mm:PinHeader_1x01_P1.00mm_Vertical, F.Cu at (85.4, 95.8)
- added J7: Vin, Connector_PinHeader_1.00mm:PinHeader_1x01_P1.00mm_Vertical, F.Cu at (85.4, 98.8)
- added J8: Vout, Connector_PinHeader_1.00mm:PinHeader_1x01_P1.00mm_Vertical, F.Cu at (85.4, 101.8)
- added J9: Masa, Connector_PinHeader_1.00mm:PinHeader_1x03_P1.00mm_Vertical, F.Cu at (88.8, 95.8)
Other:
- board text added: "Teoría de los circuitos 2 Alumnos: Alterino Perazzo, Thiago Alvarez Olmedo, Joaquín Ezequiel Montenegro, Maximiliano Ezequiel"

Commit message: actualizo desde linux
Parts:
- C1, C2, C3, C4: footprint Capacitor_THT:C_Rect_L7.2mm_W2.5mm_P5.00mm_FKS2_FKP2_MKS2_MKP2 -> Capacitor_THT:C_Rect_L11.0mm_W3.4mm_P10.00mm_MKT
- CVdd2, CVss2: footprint Capacitor_THT:C_Disc_D5.0mm_W2.5mm_P5.00mm -> Capacitor_THT:C_Disc_D5.0mm_W2.5mm_P2.50mm
- j1: footprint Connector:Banana_Cliff_FCR7350R_S16N-PC_Horizontal -> Connector:Banana_Jack_1Pin
- j2: footprint Connector:Banana_Cliff_FCR7350L_S16N-PC_Horizontal -> Connector:Banana_Jack_1Pin
- j3: footprint Connector:Banana_Cliff_FCR7350G_S16N-PC_Horizontal -> Connector:Banana_Jack_1Pin
- moved R12 133.3 mm to (51.7, 94.8), turned to 0 degrees
- moved R11 132.0 mm to (51.7, 90.8), turned to 0 degrees
- moved R15 124.1 mm to (51.7, 107.0), turned to 0 degrees
- moved R9 121.0 mm to (51.7, 82.7)
- moved R14 108.9 mm to (51.7, 102.9)
- moved R8 104.7 mm to (51.7, 78.6), turned to 0 degrees
- moved R10 102.4 mm to (51.7, 86.7)
- moved R16 99.3 mm to (51.7, 111.0)
- moved R6 98.9 mm to (51.7, 70.5)
- moved R1 98.5 mm to (51.7, 50.3), turned to 0 degrees
- moved R5 91.5 mm to (51.7, 66.5)
- moved R13 90.6 mm to (51.7, 98.9)
- moved R4 88.3 mm to (51.7, 62.4), turned to 0 degrees
- moved R2 84.7 mm to (51.7, 54.3)
- moved R7 79.1 mm to (51.7, 74.6)
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Routing:
- net Net-(U1E-V+): track 261.0 -> 0.00 mm
- net Net-(U1E-V-): track 109.4 -> 0.00 mm
- net Net-(J5-In): track 98.1 -> 0.00 mm
- net Net-(U1C-+): track 69.8 -> 0.00 mm
- net Net-(U2A--): track 62.4 -> 0.00 mm
- net Net-(J6-Pin_1): track 50.6 -> 0.00 mm
- net Net-(J7-Pin_1): track 34.8 -> 0.00 mm
- net Net-(U1A--): track 33.8 -> 0.00 mm
- net Net-(C4-Pad2): track 33.2 -> 0.00 mm
- net Net-(U2C--): track 32.7 -> 0.00 mm
- net Net-(C3-Pad2): track 22.9 -> 0.00 mm
- net Net-(C1-Pad2): track 22.6 -> 0.00 mm
- net Net-(U1B--): track 18.4 -> 0.00 mm
- net Net-(C2-Pad2): track 16.6 -> 0.00 mm
- net Net-(U2D-+): track 11.9 -> 0.00 mm
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- removed copper zone on B.Cu, net GND
Other:
- board size 93.5 x 96 mm -> 100 x 50 mm
- board text removed: "R5"

Commit message: última actualización del get, modifcación completa del pcb
Parts:
- removed J6: VA1, Connector_PinHeader_1.00mm:PinHeader_1x01_P1.00mm_Vertical
- removed J7: Vin, Connector_PinHeader_1.00mm:PinHeader_1x01_P1.00mm_Vertical
- removed J8: Vout, Connector_PinHeader_1.00mm:PinHeader_1x01_P1.00mm_Vertical
- removed J9: Masa, Connector_PinHeader_1.00mm:PinHeader_1x03_P1.00mm_Vertical
- J5, j4: footprint Connector_Coaxial:BNC_TEConnectivity_1478035_Horizontal -> Connector_Coaxial:BNC_Amphenol_B6252HB-NPP3G-50_Horizontal
- moved R14 145.6 mm to (194.8, 76.0), turned to 180 degrees
- moved R11 144.4 mm to (194.8, 71.0), turned to 180 degrees
- moved R12 144.4 mm to (193.2, 66.2), turned to 180 degrees
- moved R15 131.7 mm to (179.3, 74.5), turned to 180 degrees
- moved R16 129.8 mm to (180.5, 95.6), turned to 90 degrees
- moved R10 124.1 mm to (175.5, 95.6), turned to 90 degrees
- moved R9 118.2 mm to (169.1, 69.5)
- moved R13 115.1 mm to (159.0, 57.2)
- moved R8 105.0 mm to (155.4, 95.0)
- moved R5 96.9 mm to (144.6, 94.0), turned to 180 degrees
- moved R7 96.6 mm to (148.2, 77.6), turned to 90 degrees
- moved C4 93.6 mm to (156.0, 64.5)
- moved CVss2 90.7 mm to (174.5, 79.8)
- moved R2 82.5 mm to (130.8, 77.5), turned to 180 degrees
- moved R6 82.3 mm to (131.0, 92.5), turned to 180 degrees
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Routing:
- net Net-(U1E-V-): track 0.00 -> 214.2 mm
- net Net-(U1E-V+): track 0.00 -> 167.7 mm
- net Net-(U2A--): track 0.00 -> 92.3 mm
- net Net-(R3-Pad2): track 0.00 -> 91.4 mm
- net Net-(U2C--): track 0.00 -> 81.9 mm
- net Net-(C3-Pad2): track 0.00 -> 70.8 mm
- net Net-(J5-In): track 0.00 -> 59.0 mm
- net Net-(U1C-+): track 0.00 -> 53.5 mm
- net Net-(R10-Pad2): track 0.00 -> 47.7 mm
- net Net-(C4-Pad2): track 0.00 -> 41.9 mm
- net Net-(C2-Pad2): track 0.00 -> 39.3 mm
- net Net-(U1A--): track 0.00 -> 38.1 mm
- net Net-(j4-In): track 0.00 -> 18.5 mm
- net Net-(C1-Pad2): track 0.00 -> 18.1 mm
- net Net-(R16-Pad1): track 0.00 -> 16.4 mm
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- added copper zone on B.Cu, net GND

Commit message: version final
Routing:
- net Net-(C3-Pad2): track 70.8 -> 64.4 mm
- net Net-(U1E-V-): track 214.2 -> 208.2 mm
- net Net-(U2C--): track 81.9 -> 77.3 mm
- net GND: track 3.60 -> 0.00 mm
- net Net-(U1C-+): track 53.5 -> 50.5 mm
- net Net-(C2-Pad2): track 39.3 -> 36.5 mm
- net Net-(R10-Pad2): track 47.7 -> 45.9 mm
- net Net-(U1A--): track 38.1 -> 39.4 mm
- net Net-(J5-In): track 59.0 -> 60.2 mm
