File: laboratorio_1/Cad/laboratorio1.kicad_pcb (KiCad board)
At the start: 2 copper layers, 100 x 50 mm, 31 parts, among them J5 Output, U1 TL084, U2 TL084, j1 Vdd, j2 Vss, j3 GND, j4 Input

Commit message: agrega gitignore y elimina archivos temporales
Parts:
- moved R12 5.11 mm to (194.8, 71.1)
- moved R11 5.02 mm to (193.3, 66.2)
- moved R14 1.85 mm to (192.9, 76.0)
Connections:
- J5 pad 2: GND -> Net-(R10-Pad2)
Routing:
- net Net-(J5-In): track 60.2 -> 52.1 mm
- net Net-(R10-Pad2): track 45.9 -> 38.6 mm
- net Net-(C3-Pad2): track 64.4 -> 68.7 mm
- net Net-(U2C--): track 77.3 -> 74.6 mm
- net Net-(U1C-+): track 50.5 -> 52.0 mm
Other:
- board text added: "Bessel"
